File: Pentacube_PCB_V1.kicad_sch (KiCad schematic)
At the start: 32 parts, among them J1 Conn_01x02_Pin, J2 USB_B_Micro, J4 Conn_01x06_Pin, U2 TPS62162DSG, U3 USBLC6-2SC6, U4 W25Q128JVS, U5 STM32G474VETx, Y1 Crystal_GND24

Commit message: Add files via upload
Parts:
- added SW1: SW_Push, Button_Switch_SMD:SW_SPST_B3S-1000, symbol Switch:SW_Push
- C1, C2, C21, C3, C4, C5, C6: footprint Package_QFP:LQFP-100_14x14mm_P0.5mm -> Capacitor_SMD:C_0402_1005Metric
- C10, C9: footprint Package_QFP:LQFP-100_14x14mm_P0.5mm -> Capacitor_SMD:C_0603_1608Metric
- C11: value 1u -> 100n; footprint Package_QFP:LQFP-100_14x14mm_P0.5mm -> Capacitor_SMD:C_0402_1005Metric
- C12, C13, C24: footprint (none) -> Capacitor_SMD:C_0402_1005Metric
- C7, C8: footprint Package_QFP:LQFP-100_14x14mm_P0.5mm -> Capacitor_SMD:C_0805_2012Metric
- Cin4: renamed from Cin; footprint Package_SON:Texas_DSG0008A_WSON-8-1EP_2x2mm_P0.5mm_EP0.9x1.6mm_ThermalVias -> Capacitor_SMD:C_0805_2012Metric
- Cout4: renamed from Cout; footprint Package_SON:Texas_DSG0008A_WSON-8-1EP_2x2mm_P0.5mm_EP0.9x1.6mm_ThermalVias -> Capacitor_SMD:C_1206_3216Metric
- FB1, R1: footprint (none) -> Resistor_SMD:R_0402_1005Metric
- J1: footprint Button_Switch_THT:SW_NKK_GW12LJP -> Connector_PinHeader_2.54mm:PinHeader_1x02_P2.54mm_Vertical
- J2: footprint Package_DFN_QFN:WDFN-10-1EP_3x3mm_P0.5mm_EP1.8x2.5mm -> Connector_USB:USB_Micro-B_Wuerth_629105150521
- J4: footprint Button_Switch_THT:SW_NKK_GW12LJP -> Connector_PinHeader_2.54mm:PinHeader_1x06_P2.54mm_Vertical
- Lsw1: renamed from Lsw; footprint (none) -> Inductor_SMD:L_Pulse_PA4332
- R2: footprint Package_DIP:DIP-8_W7.62mm -> Resistor_SMD:R_0402_1005Metric
- Rpg1: renamed from Rpg; footprint (none) -> Resistor_SMD:R_0402_1005Metric
- U5: value STM32G474VETx -> STM32G474VET3
- Y1: footprint (none) -> Crystal:Crystal_SMD_2016-4Pin_2.0x1.6mm
Connections:
- net GND: now also SW1.1
- net NRST: now also SW1.2
- net SW_BUCK: now reaches Lsw1.1, U2.7 (SW)
Other:
- added sheet Test Points (Test_Points.kicad_sch)
- sheet Raspberry Pi CM4 ports: added +5V; removed none
- moved on the sheet: C11, J1, R1
