File: boostConverter.kicad_sch (KiCad schematic)
At the start: 34 parts, among them U11 TPS61088RHLR, U12 TPS61088RHLR

Commit message: Add files via upload
Parts:
- Cbst1, Cin2, Cin3: footprint Package_SO:TSSOP-10_3x3mm_P0.5mm -> Capacitor_SMD:C_0805_2012Metric
- Cbst2: renamed from Cbst; footprint Package_SO:TSSOP-10_3x3mm_P0.5mm -> Capacitor_SMD:C_0805_2012Metric
- Ccomp1: renamed from Ccomp; footprint Package_SO:TSSOP-10_3x3mm_P0.5mm -> Capacitor_SMD:C_0402_1005Metric
- Ccomp2, Ccomp3, Ccomp4, Css1: footprint Package_SO:TSSOP-10_3x3mm_P0.5mm -> Capacitor_SMD:C_0402_1005Metric
- Cin1, Cout1, Cout2, Cout3: footprint Package_SO:TSSOP-10_3x3mm_P0.5mm -> Capacitor_SMD:C_1210_3225Metric
- Cin5: renamed from Cin; footprint Package_SO:TSSOP-10_3x3mm_P0.5mm -> Capacitor_SMD:C_1210_3225Metric
- Cout5: renamed from Cout; footprint Package_SO:TSSOP-10_3x3mm_P0.5mm -> Capacitor_SMD:C_1210_3225Metric
- Css2: renamed from Css; footprint Package_SO:TSSOP-10_3x3mm_P0.5mm -> Capacitor_SMD:C_0402_1005Metric
- Cvcc1, Cvcc2, Cvcc3: footprint Package_SO:TSSOP-10_3x3mm_P0.5mm -> Capacitor_SMD:C_0603_1608Metric
- Cvcc4: renamed from Cvcc; footprint Package_SO:TSSOP-10_3x3mm_P0.5mm -> Capacitor_SMD:C_0603_1608Metric
- L1, L2: footprint Package_SO:SOIC-20W_7.5x12.8mm_P1.27mm -> IND_74439324015:L_Wurth_WE-XHMI-4030
- Rcomp1, Rfbt1, Rlim1, Rt1: footprint Package_DIP:DIP-8_W7.62mm -> Resistor_SMD:R_0402_1005Metric
- Rcomp2: renamed from Rcomp; footprint Package_DIP:DIP-8_W7.62mm -> Resistor_SMD:R_0402_1005Metric
- Rfbb1: footprint Package_DIP:DIP-8_W7.62mm -> Resistor_SMD:R_0805_2012Metric
- Rfbb2: renamed from Rfbb; footprint Package_DIP:DIP-8_W7.62mm -> Resistor_SMD:R_0805_2012Metric
- Rfbt2: renamed from Rfbt; footprint Package_DIP:DIP-8_W7.62mm -> Resistor_SMD:R_0402_1005Metric
- Rlim2: renamed from Rlim; footprint Package_DIP:DIP-8_W7.62mm -> Resistor_SMD:R_0402_1005Metric
- Rt2: renamed from Rt; footprint Package_DIP:DIP-8_W7.62mm -> Resistor_SMD:R_0402_1005Metric
- U11, U12: footprint TPS61088RHLR:IC_TPS61088RHLR -> TPS1088RHLR:IC_TPS61088RHLR
Connections:
- net SW_M2: now reaches Cbst1.1, L2.2, Rt1.1, U12.4 (SW_7), U12.5 (SW_4), U12.6 (SW_5), U12.7 (SW_6)
- net EN_M2: now reaches Cvcc1.1, Cvcc3.1, U12.1 (VCC), U12.2 (EN)
- net SS_M2: now reaches Css1.1, U12.10 (SS)
- net FB_M2: now reaches Rfbb1.1, Rfbt1.2, U12.17 (FB)
- net ILIM_M2: now reaches Rlim1.1, U12.19 (ILIM)
- net ILIM_M1: now reaches Rlim2.1, U11.19 (ILIM)
- net FB_M1: now reaches Rfbb2.1, Rfbt2.2, U11.17 (FB)
- net EN_M1: now reaches Cvcc2.1, Cvcc4.1, U11.1 (VCC), U11.2 (EN)
- net SS_M1: now reaches Css2.1, U11.10 (SS)
- net SW_M1: now reaches Cbst2.1, L1.2, Rt2.1, U11.4 (SW_7), U11.5 (SW_4), U11.6 (SW_5), U11.7 (SW_6)
