File: raspberryPiCM4.kicad_sch (KiCad schematic)
At the start: 0 parts

Commit message: Add files via upload
Parts:
- added C31: 47u, Capacitor_SMD:C_1210_3225Metric, symbol Device:C
- added C32, C33: 0.1u, Capacitor_SMD:C_0402_1005Metric, symbol Device:C
- added J12: Conn_01x14_Pin, Connector_PinHeader_2.54mm:PinHeader_1x14_P2.54mm_Vertical, symbol Connector:Conn_01x14_Pin
- added R20: 0.02, Resistor_SMD:R_2512_6332Metric, symbol Device:R
- added R21, R22: 10, Resistor_SMD:R_0402_1005Metric, symbol Device:R
- added R23, R24, R25: 4.7k, Resistor_SMD:R_0402_1005Metric, symbol Device:R
- added U13: INA226, Package_SO:TSSOP-10_3x3mm_P0.5mm, symbol Sensor_Energy:INA226
Connections:
- new net: C32.1, R22.1, U13.9 (Vin-)
- new net: C32.2, R21.1, U13.10 (Vin+)
- new net +3.3V: C33.1, R23.1, R24.1, R25.1, U13.1 (A1), U13.2 (A0), U13.6 (VS)
- new net +5V: C31.2, R20.1, R21.2, U13.8 (Vbus)
- new net GND: C31.1, C33.2, J12.10 (Pin_10), J12.12 (Pin_12), J12.13 (Pin_13), J12.14 (Pin_14), J12.6 (Pin_6), J12.8 (Pin_8), R20.2, R22.2, U13.7 (GND)
- new net GPIO: J12.1 (Pin_1), J12.2 (Pin_2)
- new net GPIO_PD9: R25.2, U13.3 (~{Alert})
- new net GPIO_READY: J12.4 (Pin_4)
- new net GPIO_RESET: J12.3 (Pin_3)
- new net I2C3_SCL: R24.2, U13.5 (SCL)
- new net I2C3_SDA: R23.2, U13.4 (SDA)
- new net SPI2_CS: J12.5 (Pin_5)
- new net SPI2_MISO: J12.9 (Pin_9)
- new net SPI2_MOSI: J12.11 (Pin_11)
- new net SPI2_SCLK: J12.7 (Pin_7)
